Commit message: Update robot.xacro

File: robot.xacro (robot description, xacro)
@@ -22,2 +22,15 @@
 <xacro:property name="wheel_mass" value="${wheel_density*pi_const*wheel_link_radius*wheel_link_radius*wheel_link_length}"/>
 <xacro:property name="caster_mass" value="${caster_density*(4.0/3.0)*pi_const*caster_link_radius*caster_link_radius*caster_link_radius}"/>
+<!-- Moments of inertia of the wheel -->
+<xacro:property name="Iz_wheel" value="${0.5*wheel_mass*wheel_link_radius*wheel_link_radius}"/>
+<xacro:property name="I_wheel" value="${(1.0/12.0)*wheel_mass*(3.0*wheel_link_radius*wheel_link_radius+wheel_link_length*wheel_link_length)}"/>
+<!-- Moments of inertia of the caster sphere -->
+<xacro:property name="I_caster" value="${(2.0/5.0)*caster_mass*caster_link_radius*caster_link_radius}"/>
+<!-- This macro defines the complete inertial section of the wheel -->
+<xacro:macro name="inertia_wheel">
+  <inertial>
+    <origin rpy="0 0 0" xyz="0 0 0"/>
+    <mass value="${wheel_mass}"/>
+    <inertia ixx="${I_wheel}" ixy="0.0" ixz="0.0" iyy="${I_wheel}" iyz="0" izz="${Iz_wheel}"/>
+  <inertial>
+</xacro:macro>

Commit message: Update robot.xacro

File: robot.xacro (robot description, xacro)
@@ -35,2 +35,10 @@
   <inertial>
 </xacro:macro>
+<!-- This macro defines the complete inertial section of the caster -->
+<xacro:macro name="inertia_caster">
+  <inertial>
+    <origin rpy="0 0 0" xyz="0 0 0"/>
+    <mass value="${caster_mass}"/>
+    <inertia ixx="${I_caster}" ixy="0.0" ixz="0.0" iyy="${I_caster}" iyz="0" izz="${I_caster}"/>
+  </inertial>
+</xacro:macro>

Commit message: Update robot.xacro

File: robot.xacro (robot description, xacro)
@@ -43,2 +43,33 @@
   </inertial>
 </xacro:macro>
+<!-- Over here we include the file that defines extra Gazebo options and motion control driver -->
+<xacro:include filename="$(find mobile_dd_robot)/model/robot.gazebo"/>
+<!-- We need to have this dummy link otherwise Gazebo will complain -->
+<link name="dummy">
+<\link>
+<joint name="dummy_joint" type="fixed">
+  <parent link="dummy"/>
+  <child link="body_link"/>
+</joint>
+<!-- START: Body link of the robot -->
+<link name="body_link">
+  <visual>
+    <geometry>
+      <box size="${body_link_x_dim} ${body_link_y_dim} ${body_link_z_dim}"/>
+    </geometry>
+    <origin rpy="0 0 0" xyz="0 0 0"/>
+  </visual>
+  <collision>
+    <geometry>
+      <box size="${body_link_x_dim} ${body_link_y_dim} ${body_link_z_dim}"/>
+    </geometry>
+    <origin rpy="0 0 0" xyz="0 0 0"/>
+  </collision>
+  <inertial>
+    <origin rpy="0 0 0" xyz="0 0 0"/>
+    <mass value="${body_mass}"/>
+    <inertia
+    ixx="${(1/12)*body_mass*(body_link_y_dim*body_link_y_dim+body_link_z_dim*body_link_z_dim)}" ixy="0"
+    izz="${(1/12)*body_mass*(body_link_y_dim*body_link_y_dim+body_link_x_dim*body_link_x_dim)}" />
+  </inertial>
+</link>

Commit message: Update robot.xacro

File: robot.xacro (robot description, xacro)
@@ -75,2 +75,25 @@
   </inertial>
 </link>
+<joint name="wheel1_joint" type="continuous">
+  <parent link="body_link"/>
+  <child link="wheel1_link"/>
+  <origin xyz="${-2*wheel_link_radius} ${-body_link_y_dim/2-wheel_link_length/2} ${wheel_link_z_location}" rpy="0 0 0"/>
+  <axis xyz="0 1 0"/>
+  <limit effort="1000" velocity="1000"/>
+  <dynamics damping="1.0" friction="1.0"/>
+</joint>
+<link name="wheel1_link">
+  <visual>
+    <origin rpy="1.570795 0 0" xyz="0 0 0"/>
+    <geometry>
+      <cylinder length="${wheel_link_length}" radius="${wheel_link_radius}"/>
+    </geometry>
+  </visual>
+  <collision>
+    <origin rpy="1.570795 0 0" xyz="0 0 0"/>
+    <geometry>
+      <cylinder length="${wheel_link_length}" radius="${wheel_link_radius}"/>
+    </geometry>
+  </collision>
+  <xacro:inertia_wheel/>
+</link>

Commit message: Update robot.xacro

File: robot.xacro (robot description, xacro)
@@ -1,99 +1,121 @@
 <?xml version="1.0"?>
 <robot name="differential_drive_robot" xmlns:xacro="http://www.ros.org/wiki/xacro">
-<!-- Body dimensions -->
-<xacro:property name="body_link_x_dim" value="1"/>
-<xacro:property name="body_link_y_dim" value="0.6"/>
-<xacro:property name="body_link_z_dim" value="0.3"/>
-<!-- Wheel dimensions and locations -->
-<xacro:property name="wheel_link_radius" value="0.15"/>
-<xacro:property name="wheel_link_length" value="0.1"/>
-<xacro:property name="wheel_link_z_location" value="-0.1"/>
-<!-- Caster sphere dimensions and locations -->
-<xacro:property name="caster_link_radius" value="0.15"/>
-<xacro:property name="caster_link_z_location" value="-0.1"/>
-<!-- Material density -->
-<xacro:property name="body_density" value="2710.0"/>
-<xacro:property name="wheel_density" value="2710.0"/>
-<xacro:property name="caster_density" value="2710.0"/>
-<!-- Pi constant -->
-<xacro:property name="pi_const" value="3.14159265"/>
-<!-- Robot body mass, wheel mass, caster mass -->
-<xacro:property name="body_mass" value="${body_density*body_link_x_dim*body_link_y_dim*body_link_z_dim}"/>
-<xacro:property name="wheel_mass" value="${wheel_density*pi_const*wheel_link_radius*wheel_link_radius*wheel_link_length}"/>
-<xacro:property name="caster_mass" value="${caster_density*(4.0/3.0)*pi_const*caster_link_radius*caster_link_radius*caster_link_radius}"/>
-<!-- Moments of inertia of the wheel -->
-<xacro:property name="Iz_wheel" value="${0.5*wheel_mass*wheel_link_radius*wheel_link_radius}"/>
-<xacro:property name="I_wheel" value="${(1.0/12.0)*wheel_mass*(3.0*wheel_link_radius*wheel_link_radius+wheel_link_length*wheel_link_length)}"/>
-<!-- Moments of inertia of the caster sphere -->
-<xacro:property name="I_caster" value="${(2.0/5.0)*caster_mass*caster_link_radius*caster_link_radius}"/>
-<!-- This macro defines the complete inertial section of the wheel -->
-<xacro:macro name="inertia_wheel">
-  <inertial>
-    <origin rpy="0 0 0" xyz="0 0 0"/>
-    <mass value="${wheel_mass}"/>
-    <inertia ixx="${I_wheel}" ixy="0.0" ixz="0.0" iyy="${I_wheel}" iyz="0" izz="${Iz_wheel}"/>
-  <inertial>
-</xacro:macro>
-<!-- This macro defines the complete inertial section of the caster -->
-<xacro:macro name="inertia_caster">
-  <inertial>
-    <origin rpy="0 0 0" xyz="0 0 0"/>
-    <mass value="${caster_mass}"/>
-    <inertia ixx="${I_caster}" ixy="0.0" ixz="0.0" iyy="${I_caster}" iyz="0" izz="${I_caster}"/>
-  </inertial>
-</xacro:macro>
-<!-- Over here we include the file that defines extra Gazebo options and motion control driver -->
-<xacro:include filename="$(find mobile_dd_robot)/model/robot.gazebo"/>
-<!-- We need to have this dummy link otherwise Gazebo will complain -->
-<link name="dummy">
-<\link>
-<joint name="dummy_joint" type="fixed">
-  <parent link="dummy"/>
-  <child link="body_link"/>
-</joint>
-<!-- START: Body link of the robot -->
-<link name="body_link">
-  <visual>
-    <geometry>
-      <box size="${body_link_x_dim} ${body_link_y_dim} ${body_link_z_dim}"/>
-    </geometry>
-    <origin rpy="0 0 0" xyz="0 0 0"/>
-  </visual>
-  <collision>
-    <geometry>
-      <box size="${body_link_x_dim} ${body_link_y_dim} ${body_link_z_dim}"/>
-    </geometry>
-    <origin rpy="0 0 0" xyz="0 0 0"/>
-  </collision>
-  <inertial>
-    <origin rpy="0 0 0" xyz="0 0 0"/>
-    <mass value="${body_mass}"/>
-    <inertia
-    ixx="${(1/12)*body_mass*(body_link_y_dim*body_link_y_dim+body_link_z_dim*body_link_z_dim)}" ixy="0" ixz="0"
-    iyy="${(1/12)*body_mass*(body_link_x_dim*body_link_x_dim+body_link_z_dim*body_link_z_dim)}"
-    izz="${(1/12)*body_mass*(body_link_y_dim*body_link_y_dim+body_link_x_dim*body_link_x_dim)}" />
-  </inertial>
-</link>
-<joint name="wheel1_joint" type="continuous">
-  <parent link="body_link"/>
-  <child link="wheel1_link"/>
-  <origin xyz="${-2*wheel_link_radius} ${-body_link_y_dim/2-wheel_link_length/2} ${wheel_link_z_location}" rpy="0 0 0"/>
-  <axis xyz="0 1 0"/>
-  <limit effort="1000" velocity="1000"/>
-  <dynamics damping="1.0" friction="1.0"/>
-</joint>
-<link name="wheel1_link">
-  <visual>
-    <origin rpy="1.570795 0 0" xyz="0 0 0"/>
-    <geometry>
-      <cylinder length="${wheel_link_length}" radius="${wheel_link_radius}"/>
-    </geometry>
-  </visual>
-  <collision>
-    <origin rpy="1.570795 0 0" xyz="0 0 0"/>
-    <geometry>
-      <cylinder length="${wheel_link_length}" radius="${wheel_link_radius}"/>
-    </geometry>
-  </collision>
-  <xacro:inertia_wheel/>
-</link>
+  <!-- Body dimensions -->
+  <xacro:property name="body_link_x_dim" value="1"/>
+  <xacro:property name="body_link_y_dim" value="0.6"/>
+  <xacro:property name="body_link_z_dim" value="0.3"/>
+  <!-- Wheel dimensions and locations -->
+  <xacro:property name="wheel_link_radius" value="0.15"/>
+  <xacro:property name="wheel_link_length" value="0.1"/>
+  <xacro:property name="wheel_link_z_location" value="-0.1"/>
+  <!-- Caster sphere dimensions and locations -->
+  <xacro:property name="caster_link_radius" value="0.15"/>
+  <xacro:property name="caster_link_z_location" value="-0.1"/>
+  <!-- Material density -->
+  <xacro:property name="body_density" value="2710.0"/>
+  <xacro:property name="wheel_density" value="2710.0"/>
+  <xacro:property name="caster_density" value="2710.0"/>
+  <!-- Pi constant -->
+  <xacro:property name="pi_const" value="3.14159265"/>
+  <!-- Robot body mass, wheel mass, caster mass -->
+  <xacro:property name="body_mass" value="${body_density*body_link_x_dim*body_link_y_dim*body_link_z_dim}"/>
+  <xacro:property name="wheel_mass" value="${wheel_density*pi_const*wheel_link_radius*wheel_link_radius*wheel_link_length}"/>
+  <xacro:property name="caster_mass" value="${caster_density*(4.0/3.0)*pi_const*caster_link_radius*caster_link_radius*caster_link_radius}"/>
+  <!-- Moments of inertia of the wheel -->
+  <xacro:property name="Iz_wheel" value="${0.5*wheel_mass*wheel_link_radius*wheel_link_radius}"/>
+  <xacro:property name="I_wheel" value="${(1.0/12.0)*wheel_mass*(3.0*wheel_link_radius*wheel_link_radius+wheel_link_length*wheel_link_length)}"/>
+  <!-- Moments of inertia of the caster sphere -->
+  <xacro:property name="I_caster" value="${(2.0/5.0)*caster_mass*caster_link_radius*caster_link_radius}"/>
+  <!-- This macro defines the complete inertial section of the wheel -->
+  <xacro:macro name="inertia_wheel">
+    <inertial>
+      <origin rpy="0 0 0" xyz="0 0 0"/>
+      <mass value="${wheel_mass}"/>
+      <inertia ixx="${I_wheel}" ixy="0.0" ixz="0.0" iyy="${I_wheel}" iyz="0" izz="${Iz_wheel}"/>
+    <inertial>
+  </xacro:macro>
+  <!-- This macro defines the complete inertial section of the caster -->
+  <xacro:macro name="inertia_caster">
+    <inertial>
+      <origin rpy="0 0 0" xyz="0 0 0"/>
+      <mass value="${caster_mass}"/>
+      <inertia ixx="${I_caster}" ixy="0.0" ixz="0.0" iyy="${I_caster}" iyz="0" izz="${I_caster}"/>
+    </inertial>
+  </xacro:macro>
+  <!-- Over here we include the file that defines extra Gazebo options and motion control driver -->
+  <xacro:include filename="$(find mobile_dd_robot)/model/robot.gazebo"/>
+  <!-- We need to have this dummy link otherwise Gazebo will complain -->
+  <link name="dummy">
+  <\link>
+  <joint name="dummy_joint" type="fixed">
+    <parent link="dummy"/>
+    <child link="body_link"/>
+  </joint>
+  <!-- START: Body link of the robot -->
+  <link name="body_link">
+    <visual>
+      <geometry>
+        <box size="${body_link_x_dim} ${body_link_y_dim} ${body_link_z_dim}"/>
+      </geometry>
+      <origin rpy="0 0 0" xyz="0 0 0"/>
+    </visual>
+    <collision>
+      <geometry>
+        <box size="${body_link_x_dim} ${body_link_y_dim} ${body_link_z_dim}"/>
+      </geometry>
+      <origin rpy="0 0 0" xyz="0 0 0"/>
+    </collision>
+    <inertial>
+      <origin rpy="0 0 0" xyz="0 0 0"/>
+      <mass value="${body_mass}"/>
+      <inertia
+      ixx="${(1/12)*body_mass*(body_link_y_dim*body_link_y_dim+body_link_z_dim*body_link_z_dim)}" ixy="0" ixz="0"
+      iyy="${(1/12)*body_mass*(body_link_x_dim*body_link_x_dim+body_link_z_dim*body_link_z_dim)}"
+      izz="${(1/12)*body_mass*(body_link_y_dim*body_link_y_dim+body_link_x_dim*body_link_x_dim)}" />
+    </inertial>
+  </link>
+  <joint name="wheel1_joint" type="continuous">
+    <parent link="body_link"/>
+    <child link="wheel1_link"/>
+    <origin xyz="${-2*wheel_link_radius} ${-body_link_y_dim/2-wheel_link_length/2} ${wheel_link_z_location}" rpy="0 0 0"/>
+    <axis xyz="0 1 0"/>
+    <limit effort="1000" velocity="1000"/>
+    <dynamics damping="1.0" friction="1.0"/>
+  </joint>
+  <link name="wheel1_link">
+    <visual>
+      <origin rpy="1.570795 0 0" xyz="0 0 0"/>
+      <geometry>
+        <cylinder length="${wheel_link_length}" radius="${wheel_link_radius}"/>
+      </geometry>
+    </visual>
+    <collision>
+      <origin rpy="1.570795 0 0" xyz="0 0 0"/>
+      <geometry>
+        <cylinder length="${wheel_link_length}" radius="${wheel_link_radius}"/>
+      </geometry>
+    </collision>
+    <xacro:inertia_wheel/>
+  </link>
+  <!-- START: Caster wheel -->
+  <joint name="caster_joint" type="fixed">
+    <parent link="body_link"/>
+    <child link="caster_link"/>
+    <origin xyz="${2*caster_link_radius} 0 ${caster_link_z_location}" rpy="0 0 0"/>
+  </joint>
+  <link name="caster_link">
+    <visual>
+      <origin rpy="0 0 0" xyz="0 0 0"/>
+      <geometry>
+        <sphere radius="${caster_link_radius}"/>
+      </geometry>
+    </visual>
+    <collision>
+      <origin rpy="0 0 0" xyz="0 0 0"/>
+      <geometry>
+        <sphere radius="${caster_link_radius}"/>
+      </geometry>
+    </collision>
+    <xacro:interia_caster/>
+  </link>
+</robot>

Commit message: Update robot.xacro

File: robot.xacro (robot description, xacro)
@@ -47,5 +47,5 @@
   <!-- We need to have this dummy link otherwise Gazebo will complain -->
   <link name="dummy">
-  <\link>
+  </link>
   <joint name="dummy_joint" type="fixed">
     <parent link="dummy"/>

Commit message: Update robot.xacro

File: robot.xacro (robot description, xacro)
@@ -33,5 +33,5 @@
       <mass value="${wheel_mass}"/>
       <inertia ixx="${I_wheel}" ixy="0.0" ixz="0.0" iyy="${I_wheel}" iyz="0" izz="${Iz_wheel}"/>
-    <inertial>
+    </inertial>
   </xacro:macro>
   <!-- This macro defines the complete inertial section of the caster -->
@@ -117,5 +117,5 @@
       </geometry>
     </collision>
-    <xacro:interia_caster/>
+    <xacro:inertia_caster/>
   </link>
 </robot>

Commit message: Update robot.xacro

File: robot.xacro (robot description, xacro)
@@ -32,5 +32,5 @@
       <origin rpy="0 0 0" xyz="0 0 0"/>
       <mass value="${wheel_mass}"/>
-      <inertia ixx="${I_wheel}" ixy="0.0" ixz="0.0" iyy="${I_wheel}" iyz="0" izz="${Iz_wheel}"/>
+      <inertia ixx="${I_wheel}" ixy="0.0" ixz="0.0" iyy="${I_wheel}" iyz="0.0" izz="${Iz_wheel}"/>
     </inertial>
   </xacro:macro>
@@ -40,5 +40,5 @@
       <origin rpy="0 0 0" xyz="0 0 0"/>
       <mass value="${caster_mass}"/>
-      <inertia ixx="${I_caster}" ixy="0.0" ixz="0.0" iyy="${I_caster}" iyz="0" izz="${I_caster}"/>
+      <inertia ixx="${I_caster}" ixy="0.0" ixz="0.0" iyy="${I_caster}" iyz="0.0" izz="${I_caster}"/>
     </inertial>
   </xacro:macro>
@@ -70,7 +70,7 @@
       <mass value="${body_mass}"/>
       <inertia
-      ixx="${(1/12)*body_mass*(body_link_y_dim*body_link_y_dim+body_link_z_dim*body_link_z_dim)}" ixy="0" ixz="0"
-      iyy="${(1/12)*body_mass*(body_link_x_dim*body_link_x_dim+body_link_z_dim*body_link_z_dim)}"
-      izz="${(1/12)*body_mass*(body_link_y_dim*body_link_y_dim+body_link_x_dim*body_link_x_dim)}" />
+      ixx="${(1.0/12.0)*body_mass*(body_link_y_dim*body_link_y_dim+body_link_z_dim*body_link_z_dim)}" ixy="0" ixz="0"
+      iyy="${(1.0/12.0)*body_mass*(body_link_x_dim*body_link_x_dim+body_link_z_dim*body_link_z_dim)}"
+      izz="${(1.0/12.0)*body_mass*(body_link_y_dim*body_link_y_dim+body_link_x_dim*body_link_x_dim)}" />
     </inertial>
   </link>

Commit message: Update robot.xacro

File: robot.xacro (robot description, xacro)
@@ -98,4 +98,27 @@
     <xacro:inertia_wheel/>
   </link>
+  <joint name="wheel2_joint" type="continuous">
+    <parent link="body_link"/>
+    <child link="wheel2_link"/>
+    <origin xyz="${-2*wheel_link_radius} ${body_link_y_dim/2+wheel_link_length/2} ${wheel_link_z_location}" rpy="0 0 0"/>
+    <axis xyz="0 1 0"/>
+    <limit effort="1000" velocity="1000"/>
+    <dynamics damping="1.0" friction="1.0"/>
+  </joint>
+  <link name="wheel2_link">
+    <visual>
+      <origin rpy="1.570795 0 0" xyz="0 0 0"/>
+      <geometry>
+        <cylinder length="${wheel_link_length}" radius="${wheel_link_radius}"/>
+      </geometry>
+    </visual>
+    <collision>
+      <origin rpy="1.570795 0 0" xyz="0 0 0"/>
+      <geometry>
+        <cylinder length="${wheel_link_length}" radius="${wheel_link_radius}"/>
+      </geometry>
+    </collision>
+    <xacro:inertia_wheel/>
+  </link>
   <!-- START: Caster wheel -->
   <joint name="caster_joint" type="fixed">
